File: pcb/HackpadAllan/HackpadAllan.kicad_pcb (KiCad board)
At the start: 2 copper layers, 60.1 x 80 mm, 20 parts, among them SW1 SW_Push, SW10 RotaryEncoder_Switch, SW2 SW_Push, SW3 SW_Push, SW4 SW_Push, SW5 SW_Push, SW6 SW_Push, SW7 SW_Push, SW8 SW_Push, SW9 SW_Push, U1 XIAO-RP2040-DIP

Commit message: fixed pcb, added to journal
Parts:
- D1, D2, D3, D4, D5, D6, D7, D8, D9: footprint Diode_THT:D_DO-35_SOD27_P2.54mm_Vertical_AnodeUp -> Diode_THT:D_DO-35_SOD27_P7.62mm_Horizontal
Routing:
- net Net-(D9-A): track 13.3 -> 15.4 mm
- net Net-(D7-A): track 13.3 -> 15.4 mm
- net Net-(D6-A): track 13.3 -> 15.4 mm
- net Net-(D4-A): track 13.3 -> 15.4 mm
- net Net-(D3-A): track 13.3 -> 15.4 mm
- net Net-(D1-A): track 13.3 -> 15.4 mm
- net Net-(D8-A): track 13.3 -> 15.4 mm
- net Net-(D5-A): track 13.3 -> 15.4 mm
- net Net-(D2-A): track 13.3 -> 15.4 mm
